Commit message: 11_11

File: src/kuavo_assets/models/biped_s44/urdf/drake/biped_v3.urdf (robot description, URDF)
Before this commit: robot biped_v3, 13 links, 12 joints
Links:
- link torso: mass 27.59893803 -> 33.61133803

File: src/kuavo_assets/models/biped_s44/urdf/drake/biped_v3_all_joint.urdf (robot description, URDF)
Before this commit: robot biped_v3_all_joint, 27 links, 22 joints
Links:
- link torso: mass 22.70214316 -> 23.49454316

File: src/kuavo_assets/models/biped_s44/urdf/drake/biped_v3_full.urdf (robot description, URDF)
Before this commit: robot biped_v3_full, 19 links, 18 joints
Links:
- link torso: mass 23.34493803 -> 24.13733803
